Commit message: restarted project

File: servo_controller/urdf/finalmodel.xacro (robot description, xacro)
@@ -1,10 +1,14 @@
 <?xml version="1.0" ?>
 <!-- =================================================================================== -->
-<!-- |    This document was autogenerated by xacro from fixed_urdf.urdf.xacro          | -->
+<!-- |    This document was autogenerated by xacro from /home/samee/ros2_ws/src/servo_controller/urdf/fixed_urdf2.urdf | -->
 <!-- |    EDITING THIS FILE BY HAND IS NOT RECOMMENDED                                 | -->
 <!-- =================================================================================== -->
-<robot name="robot">
+<robot xmlns:xacro="http://www.ros.org/wiki/xacro"  name="robot">
+  <!-- <link name="world"/> -->
+  <!-- <joint name="fixed" type="fixed">
+    <parent link="world"/>
+    <child link="base_link"/>
+  </joint> -->
   <link name="base_link">
-    <inertial auto="true"/>
     <visual>
       <geometry>
@@ -13,28 +17,14 @@
     </visual>
     <collision>
-      <density>1240.0</density>
       <geometry>
         <box size="0.254 0.127 0.0635"/>
       </geometry>
     </collision>
-  </link>
-  <!-- <link name="lidar_link">
-    <visual>
-      <geometry>
-        <box size="0.080 0.060 0.050"/>
-      </geometry>
-    </visual>
-    <inertial>
-      <origin xyz="0.000 0.000 0.000" rpy ="0.000 0.000 0.000"/>
-      <mass value="0.050"/>
-      <inertia ixx="0.00092" ixy="0.00000" ixz="0.00001" iyy="0.00094" iyz="0.00000" izz="0.00093"/>
-    </inertial>
-    <collision>
-      <origin xyz="0.010 0.000 -0.015" rpy ="0.000 0.000 0.000"/>
-      <geometry>
-        <box size="0.080 0.060 0.050"/>
-      </geometry>
-    </collision>
-  </link> -->
+    <inertial>
+      <origin rpy="0.000 0.000 0.000" xyz="0.000 0.000 0.000"/>
+      <mass value="2.000"/>
+      <inertia ixx="0.03562" ixy="0.00000" ixz="0.00000" iyy="0.04262" iyz="0.00000" izz="0.04508"/>
+    </inertial>
+  </link>
   <!-- FL -->
   <joint name="hip_fl" type="revolute">
@@ -45,17 +35,21 @@
   </joint>
   <link name="hipbone_fl">
-    <inertial auto="true"/>
-    <visual>
-      <origin rpy="0 0 0" xyz=" 0.0 0.0 0"/>
-      <geometry>
-        <box size="0.0635 0.03175 0.0381"/>
-      </geometry>
-    </visual>
-    <collision>
-      <origin rpy="0 0 0" xyz=" 0.0 0.0 0"/>
-      <geometry>
-        <box size="0.0635 0.03175 0.0381"/>
-      </geometry>
-    </collision>
+    <visual>
+      <origin rpy="0 0 0" xyz=" 0.0 0.0 0"/>
+      <geometry>
+        <box size="0.0635 0.03175 0.0381"/>
+      </geometry>
+    </visual>
+    <collision>
+      <origin rpy="0 0 0" xyz=" 0.0 0.0 0"/>
+      <geometry>
+        <box size="0.0635 0.03175 0.0381"/>
+      </geometry>
+    </collision>
+    <inertial>
+      <origin rpy="0.000 0.000 0.000" xyz="0.000 0.000 0.000"/>
+      <mass value="0.233"/>
+      <inertia ixx="0.00216" ixy="-0.00001" ixz="0.00001" iyy="0.00216" iyz="0.00001" izz="0.00211"/>
+    </inertial>
   </link>
   <joint name="shoulder_fl" type="revolute">
@@ -67,20 +61,24 @@
   </joint>
   <link name="femur_fl">
-    <inertial auto="true"/>
-    <visual>
-      <origin rpy="0 0 0" xyz="0.0 0.027 -0.0635"/>
-      <geometry>
-        <box size="0.0254 0.0254 0.127"/>
-      </geometry>
-    </visual>
-    <collision>
-      <origin rpy="0 0 0" xyz="0.0 0.027 -0.0635"/>
-      <geometry>
-        <box size="0.0254 0.0254 0.127"/>
-      </geometry>
-    </collision>
+    <visual>
+      <origin rpy="0 0 0" xyz="0.0 0.027 -0.0635"/>
+      <geometry>
+        <box size="0.0254 0.0254 0.127"/>
+      </geometry>
+    </visual>
+    <collision>
+      <origin rpy="0 0 0" xyz="0.0 0.027 -0.0635"/>
+      <geometry>
+        <box size="0.0254 0.0254 0.127"/>
+      </geometry>
+    </collision>
+    <inertial>
+      <origin rpy="0.000 0.000 0.000" xyz="0.000 0.000 0.000"/>
+      <mass value="0.084"/>
+      <inertia ixx="0.00414" ixy="0.00000" ixz="0.00000" iyy="0.00410" iyz="0.00006" izz="0.00386"/>
+    </inertial>
   </link>
   <joint name="knee_fl" type="revolute">
-    <limit effort="100" lower="-2" upper="-0.5" velocity="10"/>
+    <limit effort="100" lower="-2" upper="-0.4" velocity="10"/>
     <origin rpy="0 0 1.57" xyz="0 0 -0.127"/>
     <parent link="femur_fl"/>
@@ -88,17 +86,21 @@
   </joint>
   <link name="tibia_fl">
-    <inertial auto="true"/>
-    <visual>
-      <origin rpy="0 0 0" xyz="0.0254 0.0 -0.06985"/>
-      <geometry>
-        <box size="0.00635 0.00635 0.1397"/>
-      </geometry>
-    </visual>
-    <collision>
-      <origin rpy="0 0 0" xyz="0.0254 0.0 -0.06985"/>
-      <geometry>
-        <box size="0.00635 0.00635 0.1397"/>
-      </geometry>
-    </collision>
+    <visual>
+      <origin rpy="0 0 0" xyz="0.0254 0.0 -0.06985"/>
+      <geometry>
+        <box size="0.00635 0.00635 0.1397"/>
+      </geometry>
+    </visual>
+    <collision>
+      <origin rpy="0 0 0" xyz="0.0254 0.0 -0.06985"/>
+      <geometry>
+        <box size="0.00635 0.00635 0.1397"/>
+      </geometry>
+    </collision>
+    <inertial>
+      <origin rpy="0.000 0.000 0.000" xyz="0.000 0.000 0.000"/>
+      <mass value="0.034"/>
+      <inertia ixx="0.00159" ixy="0.00000" ixz="-0.00001" iyy="0.00159" iyz="0.00000" izz="0.00147"/>
+    </inertial>
   </link>
   <!-- FR -->
@@ -110,17 +112,21 @@
   </joint>
   <link name="hipbone_fr">
-    <inertial auto="true"/>
-    <visual>
-      <origin rpy="0 0 0" xyz=" 0.0 0.0 0"/>
-      <geometry>
-        <box size="0.0635 0.03175 0.0381"/>
-      </geometry>
-    </visual>
-    <collision>
-      <origin rpy="0 0 0" xyz=" 0.0 0.0 0"/>
-      <geometry>
-        <box size="0.0635 0.03175 0.0381"/>
-      </geometry>
-    </collision>
+    <visual>
+      <origin rpy="0 0 0" xyz=" 0.0 0.0 0"/>
+      <geometry>
+        <box size="0.0635 0.03175 0.0381"/>
+      </geometry>
+    </visual>
+    <collision>
+      <origin rpy="0 0 0" xyz=" 0.0 0.0 0"/>
+      <geometry>
+        <box size="0.0635 0.03175 0.0381"/>
+      </geometry>
+    </collision>
+    <inertial>
+      <origin rpy="0.000 0.000 0.000" xyz="0.000 0.000 0.000"/>
+      <mass value="0.233"/>
+      <inertia ixx="0.00216" ixy="0.00001" ixz="0.00001" iyy="0.00216" iyz="-0.00001" izz="0.00211"/>
+    </inertial>
   </link>
   <joint name="shoulder_fr" type="revolute">
@@ -132,17 +138,21 @@
   </joint>
   <link name="femur_fr">
-    <inertial auto="true"/>
-    <visual>
-      <origin rpy="0 0 0" xyz="0.0 0.027 -0.0635"/>
-      <geometry>
-        <box size="0.0254 0.0254 0.127"/>
-      </geometry>
-    </visual>
-    <collision>
-      <origin rpy="0 0 0" xyz="0.0 0.027 -0.0635"/>
-      <geometry>
-        <box size="0.0254 0.0254 0.127"/>
-      </geometry>
-    </collision>
+    <visual>
+      <origin rpy="0 0 0" xyz="0.0 0.027 -0.0635"/>
+      <geometry>
+        <box size="0.0254 0.0254 0.127"/>
+      </geometry>
+    </visual>
+    <collision>
+      <origin rpy="0 0 0" xyz="0.0 0.027 -0.0635"/>
+      <geometry>
+        <box size="0.0254 0.0254 0.127"/>
+      </geometry>
+    </collision>
+    <inertial>
+      <origin rpy="0.000 0.000 0.000" xyz="0.000 0.000 0.000"/>
+      <mass value="0.084"/>
+      <inertia ixx="0.00414" ixy="0.00000" ixz="0.00000" iyy="0.00410" iyz="-0.00006" izz="0.00386"/>
+    </inertial>
   </link>
   <joint name="knee_fr" type="revolute">
@@ -153,17 +163,21 @@
   </joint>
   <link name="tibia_fr">
-    <inertial auto="true"/>
-    <visual>
-      <origin rpy="0 0 0" xyz="0.0254 0.0 -0.06985"/>
-      <geometry>
-        <box size="0.00635 0.00635 0.1397"/>
-      </geometry>
-    </visual>
-    <collision>
-      <origin rpy="0 0 0" xyz="0.0254 0.0 -0.06985"/>
-      <geometry>
-        <box size="0.00635 0.00635 0.1397"/>
-      </geometry>
-    </collision>
+    <visual>
+      <origin rpy="0 0 0" xyz="0.0254 0.0 -0.06985"/>
+      <geometry>
+        <box size="0.00635 0.00635 0.1397"/>
+      </geometry>
+    </visual>
+    <collision>
+      <origin rpy="0 0 0" xyz="0.0254 0.0 -0.06985"/>
+      <geometry>
+        <box size="0.00635 0.00635 0.1397"/>
+      </geometry>
+    </collision>
+    <inertial>
+      <origin rpy="0.000 0.000 0.000" xyz="0.000 0.000 0.000"/>
+      <mass value="0.034"/>
+      <inertia ixx="0.00159" ixy="0.00000" ixz="-0.00001" iyy="0.00159" iyz="0.00000" izz="0.00147"/>
+    </inertial>
   </link>
   <!-- BR -->
@@ -175,17 +189,21 @@
   </joint>
   <link name="hipbone_br">
-    <inertial auto="true"/>
-    <visual>
-      <origin rpy="0 0 0" xyz=" 0.0 0.0 0"/>
-      <geometry>
-        <box size="0.0635 0.03175 0.0381"/>
-      </geometry>
-    </visual>
-    <collision>
-      <origin rpy="0 0 0" xyz=" 0.0 0.0 0"/>
-      <geometry>
-        <box size="0.0635 0.03175 0.0381"/>
-      </geometry>
-    </collision>
+    <visual>
+      <origin rpy="0 0 0" xyz=" 0.0 0.0 0"/>
+      <geometry>
+        <box size="0.0635 0.03175 0.0381"/>
+      </geometry>
+    </visual>
+    <collision>
+      <origin rpy="0 0 0" xyz=" 0.0 0.0 0"/>
+      <geometry>
+        <box size="0.0635 0.03175 0.0381"/>
+      </geometry>
+    </collision>
+    <inertial>
+      <origin rpy="0.000 0.000 0.000" xyz="0.000 0.000 0.000"/>
+      <mass value="0.233"/>
+      <inertia ixx="0.00216" ixy="-0.00001" ixz="-0.00001" iyy="0.00216" iyz="-0.00001" izz="0.00211"/>
+    </inertial>
   </link>
   <joint name="shoulder_br" type="revolute">
@@ -197,17 +215,21 @@
   </joint>
   <link name="femur_br">
-    <inertial auto="true"/>
-    <visual>
-      <origin rpy="0 0 0" xyz="0.0 0.027 -0.0635"/>
-      <geometry>
-        <box size="0.0254 0.0254 0.127"/>
-      </geometry>
-    </visual>
-    <collision>
-      <origin rpy="0 0 0" xyz="0.0 0.027 -0.0635"/>
-      <geometry>
-        <box size="0.0254 0.0254 0.127"/>
-      </geometry>
-    </collision>
+    <visual>
+      <origin rpy="0 0 0" xyz="0.0 0.027 -0.0635"/>
+      <geometry>
+        <box size="0.0254 0.0254 0.127"/>
+      </geometry>
+    </visual>
+    <collision>
+      <origin rpy="0 0 0" xyz="0.0 0.027 -0.0635"/>
+      <geometry>
+        <box size="0.0254 0.0254 0.127"/>
+      </geometry>
+    </collision>
+    <inertial>
+      <origin rpy="0.000 0.000 0.000" xyz="0.000 0.000 0.000"/>
+      <mass value="0.084"/>
+      <inertia ixx="0.00414" ixy="0.00000" ixz="0.00000" iyy="0.00410" iyz="-0.00006" izz="0.00386"/>
+    </inertial>
   </link>
   <joint name="knee_br" type="revolute">
@@ -218,21 +240,24 @@
   </joint>
   <link name="tibia_br">
-    <inertial auto="true"/>
-    <visual>
-      <origin rpy="0 0 0" xyz="0.0254 0.0 -0.06985"/>
-      <geometry>
-        <box size="0.00635 0.00635 0.1397"/>
-      </geometry>
-    </visual>
-    <collision>
-      <origin rpy="0 0 0" xyz="0.0254 0.0 -0.06985"/>
-      <geometry>
-        <box size="0.00635 0.00635 0.1397"/>
-      </geometry>
-    </collision>
+    <visual>
+      <origin rpy="0 0 0" xyz="0.0254 0.0 -0.06985"/>
+      <geometry>
+        <box size="0.00635 0.00635 0.1397"/>
+      </geometry>
+    </visual>
+    <collision>
+      <origin rpy="0 0 0" xyz="0.0254 0.0 -0.06985"/>
+      <geometry>
+        <box size="0.00635 0.00635 0.1397"/>
+      </geometry>
+    </collision>
+    <inertial>
+      <origin rpy="0.000 0.000 0.000" xyz="0.000 0.000 0.000"/>
+      <mass value="0.034"/>
+      <inertia ixx="0.00159" ixy="0.00000" ixz="-0.00001" iyy="0.00159" iyz="0.00000" izz="0.00147"/>
+    </inertial>
   </link>
   <!-- BL -->
   <joint name="hip_bl" type="revolute">
-    ]
     <limit effort="100" lower="-0.2" upper="0.4" velocity="10"/>
     <origin rpy="0 0 0" xyz="-0.0508 0.0508 0"/>
@@ -241,17 +266,21 @@
   </joint>
   <link name="hipbone_bl">
-    <inertial auto="true"/>
-    <visual>
-      <origin rpy="0 0 0" xyz=" 0.0 0.0 0"/>
-      <geometry>
-        <box size="0.0635 0.03175 0.0381"/>
-      </geometry>
-    </visual>
-    <collision>
-      <origin rpy="0 0 0" xyz=" 0.0 0.0 0"/>
-      <geometry>
-        <box size="0.0635 0.03175 0.0381"/>
-      </geometry>
-    </collision>
+    <visual>
+      <origin rpy="0 0 0" xyz=" 0.0 0.0 0"/>
+      <geometry>
+        <box size="0.0635 0.03175 0.0381"/>
+      </geometry>
+    </visual>
+    <collision>
+      <origin rpy="0 0 0" xyz=" 0.0 0.0 0"/>
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
File: servo_controller/urdf/fixed_urdf.urdf (robot description, URDF)
Before this commit: robot robot, 13 links, 12 joints
Links:
- added link world
Joints:
- added joint fixed: type fixed, parent world, child base_link
