Commit message: added gazebo controller

File: servo_controller/urdf/ros2control_old.urdf.xacro (robot description, xacro)
@@ -4,9 +4,10 @@
 <!-- |    EDITING THIS FILE BY HAND IS NOT RECOMMENDED                                 | -->
 <!-- =================================================================================== -->
-<robot xmlns:xacro="http://www.ros.org/wiki/xacro" name="robot">
+<robot xmlns:xacro="http://www.ros.org/wiki/xacro"  name="robot">
   <!-- Gazebo plugin for ros2_control -->
   <gazebo>
     <plugin name="gazebo_ros2_control" filename="libgazebo_ros2_control.so">
       <parameters>$(find servo_controller)/config/robot_controllers.yaml</parameters>
+      <robotNamespace>/</robotNamespace>
     </plugin>
   </gazebo>
@@ -34,15 +35,25 @@
     <parent link="base_link"/>
     <child link="hipbone_fl"/>
-    <axis xyz="0 1 0"/>
+    <!-- ros2_control Transmission -->
+    <transmission>
+      <type>transmission_interface/SimpleTransmission</type>
+      <joint name="hip_fl">
+        <hardwareInterface>hardware_interface/PositionJointInterface</hardwareInterface>
+      </joint>
+      <actuator name="hip_fl_motor">
+        <hardwareInterface>hardware_interface/PositionJointInterface</hardwareInterface>
+        <mechanicalReduction>1</mechanicalReduction>
+      </actuator>
+    </transmission>
   </joint>
   <link name="hipbone_fl">
     <visual>
-      <origin rpy="0 0 0" xyz="0.0 0.0 0"/>
-      <geometry>
-        <box size="0.0635 0.03175 0.0381"/>
-      </geometry>
-    </visual>
-    <collision>
-      <origin rpy="0 0 0" xyz="0.0 0.0 0"/>
+      <origin rpy="0 0 0" xyz=" 0.0 0.0 0"/>
+      <geometry>
+        <box size="0.0635 0.03175 0.0381"/>
+      </geometry>
+    </visual>
+    <collision>
+      <origin rpy="0 0 0" xyz=" 0.0 0.0 0"/>
       <geometry>
         <box size="0.0635 0.03175 0.0381"/>
@@ -61,4 +72,15 @@
     <parent link="hipbone_fl"/>
     <child link="femur_fl"/>
+    <!-- ros2_control Transmission -->
+    <transmission>
+      <type>transmission_interface/SimpleTransmission</type>
+      <joint name="shoulder_fl">
+        <hardwareInterface>hardware_interface/PositionJointInterface</hardwareInterface>
+      </joint>
+      <actuator name="shoulder_fl_motor">
+        <hardwareInterface>hardware_interface/PositionJointInterface</hardwareInterface>
+        <mechanicalReduction>1</mechanicalReduction>
+      </actuator>
+    </transmission>
   </joint>
   <link name="femur_fl">
@@ -86,4 +108,15 @@
     <parent link="femur_fl"/>
     <child link="tibia_fl"/>
+    <!-- ros2_control Transmission -->
+    <transmission>
+      <type>transmission_interface/SimpleTransmission</type>
+      <joint name="knee_fl">
+        <hardwareInterface>hardware_interface/PositionJointInterface</hardwareInterface>
+      </joint>
+      <actuator name="knee_fl_motor">
+        <hardwareInterface>hardware_interface/PositionJointInterface</hardwareInterface>
+        <mechanicalReduction>1</mechanicalReduction>
+      </actuator>
+    </transmission>
   </joint>
   <link name="tibia_fl">
@@ -112,5 +145,15 @@
     <parent link="base_link"/>
     <child link="hipbone_fr"/>
-    <axis xyz="0 1 0"/>
+    <!-- ros2_control Transmission -->
+    <transmission>
+      <type>transmission_interface/SimpleTransmission</type>
+      <joint name="hip_fr">
+        <hardwareInterface>hardware_interface/PositionJointInterface</hardwareInterface>
+      </joint>
+      <actuator name="hip_fr_motor">
+        <hardwareInterface>hardware_interface/PositionJointInterface</hardwareInterface>
+        <mechanicalReduction>1</mechanicalReduction>
+      </actuator>
+    </transmission>
   </joint>
   <link name="hipbone_fr">
@@ -139,4 +182,15 @@
     <parent link="hipbone_fr"/>
     <child link="femur_fr"/>
+    <!-- ros2_control Transmission -->
+    <transmission>
+      <type>transmission_interface/SimpleTransmission</type>
+      <joint name="shoulder_fr">
+        <hardwareInterface>hardware_interface/PositionJointInterface</hardwareInterface>
+      </joint>
+      <actuator name="shoulder_fr_motor">
+        <hardwareInterface>hardware_interface/PositionJointInterface</hardwareInterface>
+        <mechanicalReduction>1</mechanicalReduction>
+      </actuator>
+    </transmission>
   </joint>
   <link name="femur_fr">
@@ -164,4 +218,15 @@
     <parent link="femur_fr"/>
     <child link="tibia_fr"/>
+    <!-- ros2_control Transmission -->
+    <transmission>
+      <type>transmission_interface/SimpleTransmission</type>
+      <joint name="knee_fr">
+        <hardwareInterface>hardware_interface/PositionJointInterface</hardwareInterface>
+      </joint>
+      <actuator name="knee_fr_motor">
+        <hardwareInterface>hardware_interface/PositionJointInterface</hardwareInterface>
+        <mechanicalReduction>1</mechanicalReduction>
+      </actuator>
+    </transmission>
   </joint>
   <link name="tibia_fr">
@@ -190,5 +255,15 @@
     <parent link="base_link"/>
     <child link="hipbone_br"/>
-    <axis xyz="0 1 0"/>
+    <!-- ros2_control Transmission -->
+    <transmission>
+      <type>transmission_interface/SimpleTransmission</type>
+      <joint name="hip_br">
+        <hardwareInterface>hardware_interface/PositionJointInterface</hardwareInterface>
+      </joint>
+      <actuator name="hip_br_motor">
+        <hardwareInterface>hardware_interface/PositionJointInterface</hardwareInterface>
+        <mechanicalReduction>1</mechanicalReduction>
+      </actuator>
+    </transmission>
   </joint>
   <link name="hipbone_br">
@@ -217,4 +292,15 @@
     <parent link="hipbone_br"/>
     <child link="femur_br"/>
+    <!-- ros2_control Transmission -->
+    <transmission>
+      <type>transmission_interface/SimpleTransmission</type>
+      <joint name="shoulder_br">
+        <hardwareInterface>hardware_interface/PositionJointInterface</hardwareInterface>
+      </joint>
+      <actuator name="shoulder_br_motor">
+        <hardwareInterface>hardware_interface/PositionJointInterface</hardwareInterface>
+        <mechanicalReduction>1</mechanicalReduction>
+      </actuator>
+    </transmission>
   </joint>
   <link name="femur_br">
@@ -242,4 +328,15 @@
     <parent link="femur_br"/>
     <child link="tibia_br"/>
+    <!-- ros2_control Transmission -->
+    <transmission>
+      <type>transmission_interface/SimpleTransmission</type>
+      <joint name="knee_br">
+        <hardwareInterface>hardware_interface/PositionJointInterface</hardwareInterface>
+      </joint>
+      <actuator name="knee_br_motor">
+        <hardwareInterface>hardware_interface/PositionJointInterface</hardwareInterface>
+        <mechanicalReduction>1</mechanicalReduction>
+      </actuator>
+    </transmission>
   </joint>
   <link name="tibia_br">
@@ -268,5 +365,15 @@
     <parent link="base_link"/>
     <child link="hipbone_bl"/>
-    <axis xyz="0 1 0"/>
+    <!-- ros2_control Transmission -->
+    <transmission>
+      <type>transmission_interface/SimpleTransmission</type>
+      <joint name="hip_bl">
+        <hardwareInterface>hardware_interface/PositionJointInterface</hardwareInterface>
+      </joint>
+      <actuator name="hip_bl_motor">
+        <hardwareInterface>hardware_interface/PositionJointInterface</hardwareInterface>
+        <mechanicalReduction>1</mechanicalReduction>
+      </actuator>
+    </transmission>
   </joint>
   <link name="hipbone_bl">
@@ -295,4 +402,15 @@
     <parent link="hipbone_bl"/>
     <child link="femur_bl"/>
+    <!-- ros2_control Transmission -->
+    <transmission>
+      <type>transmission_interface/SimpleTransmission</type>
+      <joint name="shoulder_bl">
+        <hardwareInterface>hardware_interface/PositionJointInterface</hardwareInterface>
+      </joint>
+      <actuator name="shoulder_bl_motor">
+        <hardwareInterface>hardware_interface/PositionJointInterface</hardwareInterface>
+        <mechanicalReduction>1</mechanicalReduction>
+      </actuator>
+    </transmission>
   </joint>
   <link name="femur_bl">
@@ -320,4 +438,15 @@
     <parent link="femur_bl"/>
     <child link="tibia_bl"/>
+    <!-- ros2_control Transmission -->
+    <transmission>
+      <type>transmission_interface/SimpleTransmission</type>
+      <joint name="knee_bl">
+        <hardwareInterface>hardware_interface/PositionJointInterface</hardwareInterface>
+      </joint>
+      <actuator name="knee_bl_motor">
+        <hardwareInterface>hardware_interface/PositionJointInterface</hardwareInterface>
+        <mechanicalReduction>1</mechanicalReduction>
+      </actuator>
+    </transmission>
   </joint>
   <link name="tibia_bl">
@@ -340,59 +469,4 @@
     </inertial>
   </link>
-  <!-- ros2_control Configuration -->
-  <ros2_control name="GazeboSystem" type="system">
-    <hardware>
-      <plugin>gazebo_ros2_control/GazeboSystem</plugin>
-    </hardware>
-    <!-- Define all the joints that will be controlled -->
-    <joint name="hip_fl">
-      <state_interface name="position"/>
-      <command_interface name="position"/>
-    </joint>
-    <joint name="shoulder_fl">
-      <state_interface name="position"/>
-      <command_interface name="position"/>
-    </joint>
-    <joint name="knee_fl">
-      <state_interface name="position"/>
-      <command_interface name="position"/>
-    </joint>
-    <joint name="hip_fr">
-      <state_interface name="position"/>
-      <command_interface name="position"/>
-    </joint>
-    <joint name="shoulder_fr">
-      <state_interface name="position"/>
-      <command_interface name="position"/>
-    </joint>
-    <joint name="knee_fr">
-      <state_interface name="position"/>
-      <command_interface name="position"/>
-    </joint>
-    <joint name="hip_br">
-      <state_interface name="position"/>
-      <command_interface name="position"/>
-    </joint>
-    <joint name="shoulder_br">
-      <state_interface name="position"/>
-      <command_interface name="position"/>
-    </joint>
-    <joint name="knee_br">
-      <state_interface name="position"/>
-      <command_interface name="position"/>
-    </joint>
-    <joint name="hip_bl">
-      <state_interface name="position"/>
-      <command_interface name="position"/>
-    </joint>
-    <joint name="shoulder_bl">
-      <state_interface name="position"/>
-      <command_interface name="position"/>
-    </joint>
-    <joint name="knee_bl">
-      <state_interface name="position"/>
-      <command_interface name="position"/>
-    </joint>
-  </ros2_control>
-  <!-- <xacro:include filename="example_gazebo.xacro" /> -->
+  <xacro:include filename="example_gazebo.xacro" />
 </robot>
