Commit message: cleaned up repo

File: servo_controller/urdf/ros2control.urdf.xacro (robot description, xacro)
@@ -34,5 +34,5 @@
     <parent link="base_link"/>
     <child link="hipbone_fl"/>
-    <axis xyz="0 1 0"/>
+    <axis xyz="1 0 0"/>
   </joint>
   <link name="hipbone_fl">
@@ -56,5 +56,5 @@
   </link>
   <joint name="shoulder_fl" type="revolute">
-    <limit effort="100" lower="-0.1" upper="0.5" velocity="10"/>
+    <limit effort="100" lower="-0.1" upper="0.6" velocity="10"/>
     <origin rpy="0 0 0" xyz="0 0 0"/>
     <axis xyz="0 1 0"/>
@@ -82,5 +82,5 @@
   </link>
   <joint name="knee_fl" type="revolute">
-    <limit effort="100" lower="-2" upper="-0.4" velocity="10"/>
+    <limit effort="100" lower="-0.5" upper="2" velocity="10"/>
     <origin rpy="0 0 1.57" xyz="0 0 -0.127"/>
     <parent link="femur_fl"/>
@@ -112,5 +112,5 @@
     <parent link="base_link"/>
     <child link="hipbone_fr"/>
-    <axis xyz="0 1 0"/>
+    <axis xyz="1 0 0"/>
   </joint>
   <link name="hipbone_fr">
@@ -134,5 +134,5 @@
   </link>
   <joint name="shoulder_fr" type="revolute">
-    <limit effort="100" lower="-0.5" upper="0.1" velocity="10"/>
+    <limit effort="100" lower="-0.6" upper="0.1" velocity="10"/>
     <origin rpy="0 0 0" xyz="0 0 0"/>
     <axis xyz="0 1 0"/>
@@ -190,5 +190,5 @@
     <parent link="base_link"/>
     <child link="hipbone_br"/>
-    <axis xyz="0 1 0"/>
+    <axis xyz="1 0 0"/>
   </joint>
   <link name="hipbone_br">
@@ -212,5 +212,5 @@
   </link>
   <joint name="shoulder_br" type="revolute">
-    <limit effort="100" lower="-0.5" upper="0.1" velocity="10"/>
+    <limit effort="100" lower="-0.6" upper="0.1" velocity="10"/>
     <origin rpy="0 0 0" xyz="0 0 0"/>
     <axis xyz="0 1 0"/>
@@ -268,5 +268,5 @@
     <parent link="base_link"/>
     <child link="hipbone_bl"/>
-    <axis xyz="0 1 0"/>
+    <axis xyz="1 0 0"/>
   </joint>
   <link name="hipbone_bl">
@@ -290,5 +290,5 @@
   </link>
   <joint name="shoulder_bl" type="revolute">
-    <limit effort="100" lower="-0.1" upper="0.5" velocity="10"/>
+    <limit effort="100" lower="-0.1" upper="0.6" velocity="10"/>
     <origin rpy="0 0 0" xyz="0 0 0"/>
     <axis xyz="0 1 0"/>
@@ -316,5 +316,5 @@
   </link>
   <joint name="knee_bl" type="revolute">
-    <limit effort="100" lower="-2" upper="-0.4" velocity="10"/>
+    <limit effort="100" lower="-0.5" upper="2" velocity="10"/>
     <origin rpy="0 0 1.57" xyz="0 0 -0.127"/>
     <parent link="femur_bl"/>

File: servo_controller/urdf/ros2controlurdf.urdf (robot description, URDF)
Before this commit: robot robot, 13 links, 12 joints
Joints:
- joint hip_bl: axis (none) -> 0 1 0
- joint hip_br: axis (none) -> 0 1 0
- joint hip_fl: axis (none) -> 0 1 0
- joint hip_fr: axis (none) -> 0 1 0
- joint knee_bl: limit lower=-2 upper=-0.4 effort=100 velocity=10 -> lower=-0.5 upper=2 effort=100 velocity=10
- joint knee_fl: limit lower=-2 upper=-0.4 effort=100 velocity=10 -> lower=-0.5 upper=2 effort=100 velocity=10
