Commit message: last update

File: servo_controller/urdf/fixed_urdf2 old mass values.urdf (robot description, URDF)
Before this commit: robot robot, 13 links, 12 joints
Links:
- link femur_bl: mass 1 -> 0.084
- link femur_br: mass 1 -> 0.084
- link femur_fl: mass 1 -> 0.084
- link femur_fr: mass 1 -> 0.084
- link tibia_bl: mass 1 -> 0.034
- link tibia_br: mass 1 -> 0.034
- link tibia_fl: mass 1 -> 0.034
- link tibia_fr: mass 1 -> 0.034

File: servo_controller/urdf/ros2control.urdf copy.xacro (robot description, xacro)
@@ -7,19 +7,8 @@
   <!-- Gazebo plugin for ros2_control -->
   <gazebo>
-    <plugin filename="gz_ros2_control-system" name="gz_ros2_control::GazeboSimROS2ControlPlugin">
-      <parameters>/home/samee/ros2_ws/src/servo_controller/config/robot_controllers.yaml</parameters>
+    <plugin name="gazebo_ros2_control" filename="libgazebo_ros2_control.so">
+      <parameters>$(find servo_controller)/config/robot_controllers.yaml</parameters>
     </plugin>
-    <!-- <plugin filename="ign_ros2_control-system" name="ign_ros2_control::IgnitionROS2ControlPlugin">
-      <parameters>/home/samee/ros2_ws/src/servo_controller/config/robot_controllers.yaml</parameters>
-    </plugin> -->
-    <robotSimType>gazebo_ros2_control/DefaultRobotHWSim</robotSimType>
-            <robot_param>robot_description</robot_param>
-            <robot_param_node>robot_state_publisher</robot_param_node>
   </gazebo>
-<link name="base_footprint" />
-<joint name="base_footprint_joint" type="fixed">
-  <parent link="base_footprint" />
-  <child link="base_link" />
-</joint>
   <link name="base_link">
     <visual>
@@ -34,12 +23,11 @@
     </collision>
     <inertial>
-      <origin rpy="0.000 0.000 0.000" xyz="0.1 0.000 0.000"/>
-      <mass value="2.500"/>
-<inertia  ixx="0.0033602083333333335" ixy="0" ixz="0" iyy="0.011424708333333334" iyz="0" izz="0.013440833333333334" />   </inertial>
+      <origin rpy="0.000 0.000 0.000" xyz="0.000 0.000 0.000"/>
+      <mass value="2.000"/>
+<inertia  ixx="0.0033602083333333335" ixy="0" ixz="0" iyy="0.011424708333333334" iyz="0" izz="0.013440833333333334" />    </inertial>
   </link>
   <!-- FL -->
   <joint name="hip_fl" type="revolute">
-          <dynamics damping="0.7" friction="1.0"/>
-    <limit effort="100" lower="-0.2" upper="0.4"  velocity="2"/>
+    <limit effort="100" lower="-0.2" upper="0.4" velocity="10"/>
     <origin rpy="0 0 0" xyz="0.0508 0.0508 0"/>
     <parent link="base_link"/>
@@ -66,6 +54,5 @@
   </link>
   <joint name="shoulder_fl" type="revolute">
-          <dynamics damping="0.7" friction="1.0"/>
-    <limit effort="100" lower="0" upper="1"  velocity="2"/>
+    <limit effort="100" lower="-0.1" upper="0.6" velocity="10"/>
     <origin rpy="0 0 0" xyz="0 0 0"/>
     <axis xyz="0 1 0"/>
@@ -88,25 +75,14 @@
     <inertial>
       <origin rpy="0.000 0.000 0.000" xyz="0.0 0.027 -0.0635"/>
-      <mass value="1"/>
-<inertia  ixx="0.0013978466666666666" ixy="0" ixz="0" iyy="0.0013978466666666666" iyz="0" izz="0.00010752666666666665" />  </inertial>
+      <mass value="0.084"/>
+<inertia  ixx="0.00011741912" ixy="0" ixz="0" iyy="0.00011741912" iyz="0" izz="9.03224e-06" />    </inertial>
   </link>
   <joint name="knee_fl" type="revolute">
-      <dynamics damping="0.7" friction="1.0"/>
-    <limit effort="100" lower="-2.5" upper="-1"  velocity="2"/>
+    <limit effort="100" lower="-0.5" upper="2" velocity="10"/>
     <origin rpy="0 0 1.57" xyz="0 0 -0.127"/>
-    <axis xyz="1 0 0"/>
+    <axis xyz="0 1 0"/>
     <parent link="femur_fl"/>
     <child link="tibia_fl"/>
   </joint>
-<gazebo reference="tibia_fl">
-  <surface>
-    <friction>
-      <ode>
-        <mu1>100.0</mu1>         <!-- Primary friction coefficient -->
-        <mu2>100.0</mu2>       <!-- Secondary friction coefficient -->
-      </ode>
-    </friction>
-  </surface>
-</gazebo>
   <link name="tibia_fl">
     <visual>
@@ -117,5 +93,4 @@
     </visual>
     <collision>
-            <contact_coefficients mu="1"/>
       <origin rpy="0 0 0" xyz="0.0254 0.0 -0.06985"/>
       <geometry>
@@ -125,11 +100,10 @@
     <inertial>
       <origin rpy="0.000 0.000 0.000" xyz="0.0254 0.0 -0.06985"/>
-      <mass value="1"/>
-<inertia  ixx="0.001629701041666666" ixy="0" ixz="0" iyy="0.001629701041666666" iyz="0" izz="6.720416666666666e-06" />   </inertial>
+      <mass value="0.034"/>
+<inertia  ixx="5.5409835416666655e-05" ixy="0" ixz="0" iyy="5.5409835416666655e-05" iyz="0" izz="2.2849416666666668e-07" />    </inertial>
   </link>
   <!-- FR -->
   <joint name="hip_fr" type="revolute">
-          <dynamics damping="0.7" friction="1.0"/>
-    <limit effort="100" lower="-0.2" upper="0.4"  velocity="2"/>
+    <limit effort="100" lower="-0.2" upper="0.4" velocity="10"/>
     <origin rpy="0 0 3.14" xyz="0.0508 -0.0508 0"/>
     <parent link="base_link"/>
@@ -153,9 +127,8 @@
       <origin rpy="0.000 0.000 0.000" xyz="0.000 0.000 0.000"/>
       <mass value="0.233"/>
-<inertia  ixx="4.775864104166667e-05" ixy="0" ixz="0" iyy="0.00010647828166666667" iyz="0" izz="9.786606770833334e-05" />  </inertial>
+<inertia  ixx="4.775864104166667e-05" ixy="0" ixz="0" iyy="0.00010647828166666667" iyz="0" izz="9.786606770833334e-05" />    </inertial>
   </link>
   <joint name="shoulder_fr" type="revolute">
-          <dynamics damping="0.7" friction="1.0"/>
-    <limit effort="100" lower="-1" upper="0"  velocity="2"/>
+    <limit effort="100" lower="-0.6" upper="0.1" velocity="10"/>
     <origin rpy="0 0 0" xyz="0 0 0"/>
     <axis xyz="0 1 0"/>
@@ -178,25 +151,14 @@
     <inertial>
       <origin rpy="0.000 0.000 0.000" xyz="0.0 0.027 -0.0635"/>
-      <mass value="1"/>
-<inertia  ixx="0.0013978466666666666" ixy="0" ixz="0" iyy="0.0013978466666666666" iyz="0" izz="0.00010752666666666665" />  </inertial>
+      <mass value="0.084"/>
+<inertia  ixx="0.00011741912" ixy="0" ixz="0" iyy="0.00011741912" iyz="0" izz="9.03224e-06" />    </inertial>
   </link>
   <joint name="knee_fr" type="revolute">
-      <dynamics damping="0.7" friction="1.0"/>
-    <limit effort="100" lower="1" upper="2.5"  velocity="2"/>
+    <limit effort="100" lower="-0.5" upper="2" velocity="10"/>
     <origin rpy="0 0 1.57" xyz="0 0 -0.127"/>
-    <axis xyz="1 0 0"/>
+    <axis xyz="0 1 0"/>
     <parent link="femur_fr"/>
     <child link="tibia_fr"/>
   </joint>
-<gazebo reference="tibia_fr">
-  <surface>
-    <friction>
-      <ode>
-        <mu1>100.0</mu1>         <!-- Primary friction coefficient -->
-        <mu2>100.0</mu2>       <!-- Secondary friction coefficient -->
-      </ode>
-    </friction>
-  </surface>
-</gazebo>
   <link name="tibia_fr">
     <visual>
@@ -207,5 +169,4 @@
     </visual>
     <collision>
-            <contact_coefficients mu="1"/>
       <origin rpy="0 0 0" xyz="0.0254 0.0 -0.06985"/>
       <geometry>
@@ -215,11 +176,10 @@
     <inertial>
       <origin rpy="0.000 0.000 0.000" xyz="0.0254 0.0 -0.06985"/>
-      <mass value="1"/>
-<inertia  ixx="0.001629701041666666" ixy="0" ixz="0" iyy="0.001629701041666666" iyz="0" izz="6.720416666666666e-06" />   </inertial>
+      <mass value="0.034"/>
+<inertia  ixx="5.5409835416666655e-05" ixy="0" ixz="0" iyy="5.5409835416666655e-05" iyz="0" izz="2.2849416666666668e-07" />    </inertial>
   </link>
   <!-- BR -->
   <joint name="hip_br" type="revolute">
-          <dynamics damping="0.7" friction="1.0"/>
-    <limit effort="100" lower="-0.2" upper="0.4"  velocity="2"/>
+    <limit effort="100" lower="-0.2" upper="0.4" velocity="10"/>
     <origin rpy="0 0 3.14" xyz="-0.0508 -0.0508 0"/>
     <parent link="base_link"/>
@@ -243,9 +203,8 @@
       <origin rpy="0.000 0.000 0.000" xyz="0.000 0.000 0.000"/>
       <mass value="0.233"/>
-<inertia  ixx="4.775864104166667e-05" ixy="0" ixz="0" iyy="0.00010647828166666667" iyz="0" izz="9.786606770833334e-05" />   </inertial>
+<inertia  ixx="4.775864104166667e-05" ixy="0" ixz="0" iyy="0.00010647828166666667" iyz="0" izz="9.786606770833334e-05" />    </inertial>
   </link>
   <joint name="shoulder_br" type="revolute">
-          <dynamics damping="0.7" friction="1.0"/>
-    <limit effort="100" lower="-1" upper="0"  velocity="2"/>
+    <limit effort="100" lower="-0.6" upper="0.1" velocity="10"/>
     <origin rpy="0 0 0" xyz="0 0 0"/>
     <axis xyz="0 1 0"/>
@@ -268,25 +227,14 @@
     <inertial>
       <origin rpy="0.000 0.000 0.000" xyz="0.0 0.027 -0.0635"/>
-      <mass value="1"/>
-<inertia  ixx="0.0013978466666666666" ixy="0" ixz="0" iyy="0.0013978466666666666" iyz="0" izz="0.00010752666666666665" />  </inertial>
+      <mass value="0.084"/>
+<inertia  ixx="0.00011741912" ixy="0" ixz="0" iyy="0.00011741912" iyz="0" izz="9.03224e-06" />    </inertial>
   </link>
   <joint name="knee_br" type="revolute">
-      <dynamics damping="0.7" friction="1.0"/>
-    <limit effort="100" lower="1" upper="2.5"  velocity="2"/>
+    <limit effort="100" lower="-0.5" upper="2" velocity="10"/>
     <origin rpy="0 0 1.57" xyz="0 0 -0.127"/>
-    <axis xyz="1 0 0"/>
+    <axis xyz="0 1 0"/>
     <parent link="femur_br"/>
     <child link="tibia_br"/>
   </joint>
-<gazebo reference="tibia_br">
-  <surface>
-    <friction>
-      <ode>
-        <mu1>100.0</mu1>         <!-- Primary friction coefficient -->
-        <mu2>100.0</mu2>       <!-- Secondary friction coefficient -->
-      </ode>
-    </friction>
-  </surface>
-</gazebo>
   <link name="tibia_br">
     <visual>
@@ -297,5 +245,4 @@
     </visual>
     <collision>
-            <contact_coefficients mu="1"/>
       <origin rpy="0 0 0" xyz="0.0254 0.0 -0.06985"/>
       <geometry>
@@ -305,11 +252,10 @@
     <inertial>
       <origin rpy="0.000 0.000 0.000" xyz="0.0254 0.0 -0.06985"/>
-      <mass value="1"/>
-<inertia  ixx="0.001629701041666666" ixy="0" ixz="0" iyy="0.001629701041666666" iyz="0" izz="6.720416666666666e-06" />  </inertial>
+      <mass value="0.034"/>
+<inertia  ixx="5.5409835416666655e-05" ixy="0" ixz="0" iyy="5.5409835416666655e-05" iyz="0" izz="2.2849416666666668e-07" />    </inertial>
   </link>
   <!-- BL -->
   <joint name="hip_bl" type="revolute">
-          <dynamics damping="0.7" friction="1.0"/>
-    <limit effort="100" lower="-0.2" upper="0.4"  velocity="2"/>
+    <limit effort="100" lower="-0.2" upper="0.4" velocity="10"/>
     <origin rpy="0 0 0" xyz="-0.0508 0.0508 0"/>
     <parent link="base_link"/>
@@ -333,9 +279,8 @@
       <origin rpy="0.000 0.000 0.000" xyz="0.000 0.000 0.000"/>
       <mass value="0.233"/>
-<inertia  ixx="4.775864104166667e-05" ixy="0" ixz="0" iyy="0.00010647828166666667" iyz="0" izz="9.786606770833334e-05" />   </inertial>
+<inertia  ixx="4.775864104166667e-05" ixy="0" ixz="0" iyy="0.00010647828166666667" iyz="0" izz="9.786606770833334e-05" />    </inertial>
   </link>
   <joint name="shoulder_bl" type="revolute">
-          <dynamics damping="0.7" friction="1.0"/>
-    <limit effort="100" lower="0" upper="1"  velocity="2"/>
+    <limit effort="100" lower="-0.1" upper="0.6" velocity="10"/>
     <origin rpy="0 0 0" xyz="0 0 0"/>
     <axis xyz="0 1 0"/>
@@ -358,25 +303,14 @@
     <inertial>
       <origin rpy="0.000 0.000 0.000" xyz="0.0 0.027 -0.0635"/>
-      <mass value="1"/>
-<inertia  ixx="0.0013978466666666666" ixy="0" ixz="0" iyy="0.0013978466666666666" iyz="0" izz="0.00010752666666666665" /> </inertial>
+      <mass value="0.084"/>
+<inertia  ixx="0.00011741912" ixy="0" ixz="0" iyy="0.00011741912" iyz="0" izz="9.03224e-06" />    </inertial>
   </link>
   <joint name="knee_bl" type="revolute">
-      <dynamics damping="0.7" friction="1.0"/>
-    <limit effort="100" lower="-2.5" upper="-1"  velocity="2"/>
+    <limit effort="100" lower="-0.5" upper="2" velocity="10"/>
     <origin rpy="0 0 1.57" xyz="0 0 -0.127"/>
-    <axis xyz="1 0 0"/>
+      <axis xyz="0 1 0"/>
     <parent link="femur_bl"/>
     <child link="tibia_bl"/>
   </joint>
-<gazebo reference="tibia_bl">
-  <surface>
-    <friction>
-      <ode>
-        <mu1>100.0</mu1>         <!-- Primary friction coefficient -->
-        <mu2>100.0</mu2>       <!-- Secondary friction coefficient -->
-      </ode>
-    </friction>
-  </surface>
-</gazebo>
   <link name="tibia_bl">
     <visual>
@@ -387,5 +321,4 @@
     </visual>
     <collision>
-      <contact_coefficients mu="1"/>
       <origin rpy="0 0 0" xyz="0.0254 0.0 -0.06985"/>
       <geometry>
@@ -395,12 +328,11 @@
     <inertial>
       <origin rpy="0.000 0.000 0.000" xyz="0.0254 0.0 -0.06985"/>
-      <mass value="1"/>
-<inertia  ixx="0.001629701041666666" ixy="0" ixz="0" iyy="0.001629701041666666" iyz="0" izz="6.720416666666666e-06" />  </inertial>
+      <mass value="0.034"/>
+<inertia  ixx="5.5409835416666655e-05" ixy="0" ixz="0" iyy="5.5409835416666655e-05" iyz="0" izz="2.2849416666666668e-07" />   </inertial>
   </link>
   <!-- ros2_control Configuration -->
   <ros2_control name="GazeboSystem" type="system">
     <hardware>
-          <!-- <plugin>ign_ros2_control/IgnitionSystem</plugin> -->
-    <plugin>gz_ros2_control/GazeboSimSystem</plugin>
+      <plugin>gazebo_ros2_control/GazeboSystem</plugin>
     </hardware>
     <!-- Define all the joints that will be controlled -->
